File: RemoteMaster.sch (KiCad schematic (older format))
At the start: 11 parts

Commit message: Added Refrences
Used the Netlist function in KiCAD to automatically label all the components.
Parts:
- gave numbers to parts that had none: 11
Other:
- moved on the sheet: D18, R26
Changed lines of the file:
@@
 P 6550 3150
 AR Path="/5F704554" Ref="U?"  Part="1"
-AR Path="/5F6F6591/5F704554" Ref="U?"  Part="1"
-F 0 "U?" H 7550 3537 60  0000 C CNN
+AR Path="/5F6F6591/5F704554" Ref="U5"  Part="1"
+F 0 "U5" H 7550 3537 60  0000 C CNN
 F 1 "LTC4331IUFD-PBF" H 7550 3431 60  0000 C CNN
 F 2 "QFN_20_ADI" H 7550 3390 60  0001 C CNN
@@
 P 1450 3850
 AR Path="/5F70455F" Ref="#PWR?"  Part="1"
-AR Path="/5F6F6591/5F70455F" Ref="#PWR?"  Part="1"
-F 0 "#PWR?" H 1450 3700 50  0001 C CNN
+AR Path="/5F6F6591/5F70455F" Ref="#PWR0140"  Part="1"
+F 0 "#PWR0140" H 1450 3700 50  0001 C CNN
 F 1 "+5V" H 1465 4023 50  0000 C CNN
 F 2 "" H 1450 3850 50  0001 C CNN
@@
 P 5200 4100
 AR Path="/5F704567" Ref="#PWR?"  Part="1"
-AR Path="/5F6F6591/5F704567" Ref="#PWR?"  Part="1"
-F 0 "#PWR?" H 5200 3950 50  0001 C CNN
+AR Path="/5F6F6591/5F704567" Ref="#PWR0141"  Part="1"
+F 0 "#PWR0141" H 5200 3950 50  0001 C CNN
 F 1 "+5V" H 5215 4273 50  0000 C CNN
 F 2 "" H 5200 4100 50  0001 C CNN
@@
 P 4950 4100
 AR Path="/5F70456E" Ref="R?"  Part="1"
-AR Path="/5F6F6591/5F70456E" Ref="R?"  Part="1"
-F 0 "R?" V 4745 4100 50  0000 C CNN
+AR Path="/5F6F6591/5F70456E" Ref="R25"  Part="1"
+F 0 "R25" V 4745 4100 50  0000 C CNN
 F 1 "10k" V 4836 4100 50  0000 C CNN
 F 2 "" V 4990 4090 50  0001 C CNN
@@
 P 2250 2850
 AR Path="/5F704577" Ref="U?"  Part="1"
-AR Path="/5F6F6591/5F704577" Ref="U?"  Part="1"
-F 0 "U?" H 3200 3237 60  0000 C CNN
+AR Path="/5F6F6591/5F704577" Ref="U4"  Part="1"
+F 0 "U4" H 3200 3237 60  0000 C CNN
 F 1 "MCP23017-E_SP" H 3200 3131 60  0000 C CNN
 F 2 "SPDIP28_300MC_MCH" H 3200 3090 60  0001 C CNN
@@
 P 1450 4000
 AR Path="/5F704585" Ref="#PWR?"  Part="1"
-AR Path="/5F6F6591/5F704585" Ref="#PWR?"  Part="1"
-F 0 "#PWR?" H 1450 3750 50  0001 C CNN
+AR Path="/5F6F6591/5F704585" Ref="#PWR0142"  Part="1"
+F 0 "#PWR0142" H 1450 3750 50  0001 C CNN
 F 1 "Earth" H 1450 3850 50  0001 C CNN
 F 2 "" H 1450 4000 50  0001 C CNN
@@
 P 6350 3000
 AR Path="/5F70458B" Ref="#PWR?"  Part="1"
-AR Path="/5F6F6591/5F70458B" Ref="#PWR?"  Part="1"
-F 0 "#PWR?" H 6350 2850 50  0001 C CNN
+AR Path="/5F6F6591/5F70458B" Ref="#PWR0143"  Part="1"
+F 0 "#PWR0143" H 6350 2850 50  0001 C CNN
 F 1 "+5V" V 6365 3128 50  0000 L CNN
 F 2 "" H 6350 3000 50  0001 C CNN
@@
 L Device:R_US R?
 U 1 1 5F704591
-P 5650 3550
+P 5550 3550
 AR Path="/5F704591" Ref="R?"  Part="1"
-AR Path="/5F6F6591/5F704591" Ref="R?"  Part="1"
-F 0 "R?" V 5855 3550 50  0000 C CNN
-F 1 "1.5k" V 5764 3550 50  0000 C CNN
-F 2 "" V 5690 3540 50  0001 C CNN
-F 3 "~" H 5650 3550 50  0001 C CNN
-	1    5650 3550
+AR Path="/5F6F6591/5F704591" Ref="R26"  Part="1"
+F 0 "R26" V 5755 3550 50  0000 C CNN
+F 1 "1.5k" V 5664 3550 50  0000 C CNN
+F 2 "" V 5590 3540 50  0001 C CNN
+F 3 "~" H 5550 3550 50  0001 C CNN
+	1    5550 3550
 	0    -1   -1   0
 $EndComp
@@
 L power:+5V #PWR?
 U 1 1 5F704597
-P 5400 3550
+P 5300 3550
 AR Path="/5F704597" Ref="#PWR?"  Part="1"
-AR Path="/5F6F6591/5F704597" Ref="#PWR?"  Part="1"
-F 0 "#PWR?" H 5400 3400 50  0001 C CNN
-F 1 "+5V" V 5415 3678 50  0000 L CNN
-F 2 "" H 5400 3550 50  0001 C CNN
-F 3 "" H 5400 3550 50  0001 C CNN
-	1    5400 3550
+AR Path="/5F6F6591/5F704597" Ref="#PWR0144"  Part="1"
+F 0 "#PWR0144" H 5300 3400 50  0001 C CNN
+F 1 "+5V" V 5315 3678 50  0000 L CNN
+F 2 "" H 5300 3550 50  0001 C CNN
+F 3 "" H 5300 3550 50  0001 C CNN
+	1    5300 3550
 	1    0    0    -1
 $EndComp
@@
 L Device:LED D?
 U 1 1 5F70459D
-P 5950 3550
+P 5850 3550
 AR Path="/5F70459D" Ref="D?"  Part="1"
-AR Path="/5F6F6591/5F70459D" Ref="D?"  Part="1"
-F 0 "D?" H 5943 3295 50  0000 C CNN
-F 1 "LED" H 5943 3386 50  0000 C CNN
-F 2 "" H 5950 3550 50  0001 C CNN
-F 3 "~" H 5950 3550 50  0001 C CNN
-	1    5950 3550
+AR Path="/5F6F6591/5F70459D" Ref="D18"  Part="1"
+F 0 "D18" H 5843 3295 50  0000 C CNN
+F 1 "LED" H 5843 3386 50  0000 C CNN
+F 2 "" H 5850 3550 50  0001 C CNN
+F 3 "~" H 5850 3550 50  0001 C CNN
+	1    5850 3550
 	-1   0    0    1
 $EndComp
@@
 P 5700 3900
 AR Path="/5F7045A6" Ref="R?"  Part="1"
-AR Path="/5F6F6591/5F7045A6" Ref="R?"  Part="1"
-F 0 "R?" H 5768 3946 50  0000 L CNN
+AR Path="/5F6F6591/5F7045A6" Ref="R27"  Part="1"
+F 0 "R27" H 5768 3946 50  0000 L CNN
 F 1 "2.7k" H 5768 3855 50  0000 L CNN
 F 2 "" V 5740 3890 50  0001 C CNN
@@
 P 6050 4000
 AR Path="/5F7045AC" Ref="R?"  Part="1"
-AR Path="/5F6F6591/5F7045AC" Ref="R?"  Part="1"
-F 0 "R?" H 6118 4046 50  0000 L CNN
+AR Path="/5F6F6591/5F7045AC" Ref="R28"  Part="1"
+F 0 "R28" H 6118 4046 50  0000 L CNN
 F 1 "2.7k" H 6118 3955 50  0000 L CNN
 F 2 "" V 6090 3990 50  0001 C CNN
@@
 P 5850 4400
 AR Path="/5F7045BA" Ref="#PWR?"  Part="1"
-AR Path="/5F6F6591/5F7045BA" Ref="#PWR?"  Part="1"
-F 0 "#PWR?" H 5850 4250 50  0001 C CNN
+AR Path="/5F6F6591/5F7045BA" Ref="#PWR0145"  Part="1"
+F 0 "#PWR0145" H 5850 4250 50  0001 C CNN
 F 1 "+5V" H 5865 4573 50  0000 C CNN
 F 2 "" H 5850 4400 50  0001 C CNN
@@
 P 6300 3550
 AR Path="/5F7045C4" Ref="#PWR?"  Part="1"
-AR Path="/5F6F6591/5F7045C4" Ref="#PWR?"  Part="1"
-F 0 "#PWR?" H 6300 3400 50  0001 C CNN
+AR Path="/5F6F6591/5F7045C4" Ref="#PWR0146"  Part="1"
+F 0 "#PWR0146" H 6300 3400 50  0001 C CNN
 F 1 "+5V" V 6315 3678 50  0000 L CNN
 F 2 "" H 6300 3550 50  0001 C CNN
@@
 P 9050 3750
 AR Path="/5F7045CA" Ref="#PWR?"  Part="1"
-AR Path="/5F6F6591/5F7045CA" Ref="#PWR?"  Part="1"
-F 0 "#PWR?" H 9050 3600 50  0001 C CNN
+AR Path="/5F6F6591/5F7045CA" Ref="#PWR0147"  Part="1"
+F 0 "#PWR0147" H 9050 3600 50  0001 C CNN
 F 1 "+5V" V 9065 3878 50  0000 L CNN
 F 2 "" H 9050 3750 50  0001 C CNN
@@
 P 8800 3650
 AR Path="/5F7045D0" Ref="#PWR?"  Part="1"
-AR Path="/5F6F6591/5F7045D0" Ref="#PWR?"  Part="1"
-F 0 "#PWR?" H 8800 3400 50  0001 C CNN
+AR Path="/5F6F6591/5F7045D0" Ref="#PWR0148"  Part="1"
+F 0 "#PWR0148" H 8800 3400 50  0001 C CNN
 F 1 "Earth" H 8800 3500 50  0001 C CNN
 F 2 "" H 8800 3650 50  0001 C CNN
@@
 P 6550 2750
 AR Path="/5F7045D6" Ref="C?"  Part="1"
-AR Path="/5F6F6591/5F7045D6" Ref="C?"  Part="1"
-F 0 "C?" H 6665 2796 50  0000 L CNN
+AR Path="/5F6F6591/5F7045D6" Ref="C4"  Part="1"
+F 0 "C4" H 6665 2796 50  0000 L CNN
 F 1 "4.7uF" H 6665 2705 50  0000 L CNN
 F 2 "" H 6588 2600 50  0001 C CNN
@@
 P 6350 2400
 AR Path="/5F7045DC" Ref="#PWR?"  Part="1"
-AR Path="/5F6F6591/5F7045DC" Ref="#PWR?"  Part="1"
-F 0 "#PWR?" H 6350 2150 50  0001 C CNN
+AR Path="/5F6F6591/5F7045DC" Ref="#PWR0149"  Part="1"
+F 0 "#PWR0149" H 6350 2150 50  0001 C CNN
 F 1 "GND" H 6355 2227 50  0000 C CNN
 F 2 "" H 6350 2400 50  0001 C CNN
@@
 P 5950 2750
 AR Path="/5F7045E5" Ref="C?"  Part="1"
-AR Path="/5F6F6591/5F7045E5" Ref="C?"  Part="1"
-F 0 "C?" H 6065 2796 50  0000 L CNN
+AR Path="/5F6F6591/5F7045E5" Ref="C3"  Part="1"
+F 0 "C3" H 6065 2796 50  0000 L CNN
 F 1 "1uF" H 6065 2705 50  0000 L CNN
 F 2 "" H 5988 2600 50  0001 C CNN
@@
 P 5700 2400
 AR Path="/5F7045EB" Ref="#PWR?"  Part="1"
-AR Path="/5F6F6591/5F7045EB" Ref="#PWR?"  Part="1"
-F 0 "#PWR?" H 5700 2150 50  0001 C CNN
+AR Path="/5F6F6591/5F7045EB" Ref="#PWR0150"  Part="1"
+F 0 "#PWR0150" H 5700 2150 50  0001 C CNN
 F 1 "GND" H 5705 2227 50  0000 C CNN
 F 2 "" H 5700 2400 50  0001 C CNN
@@
 P 5700 3000
 AR Path="/5F7045F2" Ref="#PWR?"  Part="1"
-AR Path="/5F6F6591/5F7045F2" Ref="#PWR?"  Part="1"
-F 0 "#PWR?" H 5700 2850 50  0001 C CNN
+AR Path="/5F6F6591/5F7045F2" Ref="#PWR0151"  Part="1"
+F 0 "#PWR0151" H 5700 2850 50  0001 C CNN
 F 1 "+5V" V 5715 3128 50  0000 L CNN
 F 2 "" H 5700 3000 50  0001 C CNN
@@
 P 1450 3150
 AR Path="/5F7045FD" Ref="J?"  Part="1"
-AR Path="/5F6F6591/5F7045FD" Ref="J?"  Part="1"
-F 0 "J?" H 1558 3631 50  0000 C CNN
+AR Path="/5F6F6591/5F7045FD" Ref="J3"  Part="1"
+F 0 "J3" H 1558 3631 50  0000 C CNN
 F 1 "Conn_01x08_Male" H 1558 3540 50  0000 C CNN
 F 2 "" H 1450 3150 50  0001 C CNN
@@
 P 4800 3250
 AR Path="/5F704603" Ref="J?"  Part="1"
-AR Path="/5F6F6591/5F704603" Ref="J?"  Part="1"
-F 0 "J?" H 4908 3731 50  0000 C CNN
+AR Path="/5F6F6591/5F704603" Ref="J4"  Part="1"
+F 0 "J4" H 4908 3731 50  0000 C CNN
 F 1 "Conn_01x08_Male" H 4908 3640 50  0000 C CNN
 F 2 "" H 4800 3250 50  0001 C CNN
@@
 P 4300 4150
 AR Path="/5F70460A" Ref="#PWR?"  Part="1"
-AR Path="/5F6F6591/5F70460A" Ref="#PWR?"  Part="1"
-F 0 "#PWR?" H 4300 4000 50  0001 C CNN
+AR Path="/5F6F6591/5F70460A" Ref="#PWR0152"  Part="1"
+F 0 "#PWR0152" H 4300 4000 50  0001 C CNN
 F 1 "+5V" H 4315 4323 50  0000 C CNN
 F 2 "" H 4300 4150 50  0001 C CNN
@@
 	6100 3650 6100 3550
 Wire Wire Line
-	5500 3550 5400 3550
+	5400 3550 5300 3550
 Wire Wire Line
 	6050 4150 6050 4400
@@
 Wire Wire Line
 	6300 3550 6400 3550
+Wire Wire Line
+	6100 3550 6000 3550
 $EndSCHEMATC
