File: localMaster.sch (KiCad schematic (older format))
At the start: 12 parts

Commit message: Added Local Master I2C Address
Local Slace LTC4331 has I2C address set to 3Eh
Connections:
- net GND: now also U?.11 (A1), U?.12 (A2)
Other:
- note added: "A1 and A2 set the I2C address. \nBoth are set to low so current \naddress is 3Eh"
Changed lines of the file:
@@
 	-1   0    0    1
 $EndComp
-Text Notes 5150 4500 0    50   ~ 0
+Text Notes 5000 4400 0    50   ~ 0
 Never let SLO pin on LTC4331 float.
 Text Notes 4800 2550 0    50   ~ 0
@@
 Text HLabel 2900 2300 2    50   Input ~ 0
 Vcc
+Wire Wire Line
+	6700 4000 6700 4100
+$Comp
+L power:GND #PWR?
+U 1 1 5F7519CB
+P 6700 4100
+AR Path="/5F7519CB" Ref="#PWR?"  Part="1"
+AR Path="/5F6BFC31/5F7519CB" Ref="#PWR?"  Part="1"
+F 0 "#PWR?" H 6700 3850 50  0001 C CNN
+F 1 "GND" V 6705 3972 50  0000 R CNN
+F 2 "" H 6700 4100 50  0001 C CNN
+F 3 "" H 6700 4100 50  0001 C CNN
+	1    6700 4100
+	1    0    0    -1
+$EndComp
+Connection ~ 6700 4100
+Text Notes 6850 4350 0    50   ~ 0
+A1 and A2 set the I2C address. \nBoth are set to low so current \naddress is 3Eh
 $EndSCHEMATC

Commit message: Added Refrences
Used the Netlist function in KiCAD to automatically label all the components.
Parts:
- gave numbers to parts that had none: 12
Changed lines of the file:
@@
 P 2350 4400
 AR Path="/5F6CC2A9" Ref="#PWR?"  Part="1"
-AR Path="/5F6BFC31/5F6CC2A9" Ref="#PWR?"  Part="1"
-F 0 "#PWR?" H 2350 4150 50  0001 C CNN
+AR Path="/5F6BFC31/5F6CC2A9" Ref="#PWR0125"  Part="1"
+F 0 "#PWR0125" H 2350 4150 50  0001 C CNN
 F 1 "GND" H 2355 4227 50  0000 C CNN
 F 2 "" H 2350 4400 50  0001 C CNN
@@
 P 4600 4150
 AR Path="/5F6CC2B8" Ref="R?"  Part="1"
-AR Path="/5F6BFC31/5F6CC2B8" Ref="R?"  Part="1"
-F 0 "R?" H 4668 4196 50  0000 L CNN
+AR Path="/5F6BFC31/5F6CC2B8" Ref="R21"  Part="1"
+F 0 "R21" H 4668 4196 50  0000 L CNN
 F 1 "10k" H 4668 4105 50  0000 L CNN
 F 2 "" V 4640 4140 50  0001 C CNN
@@
 P 3850 3850
 AR Path="/5F6CC2BE" Ref="R?"  Part="1"
-AR Path="/5F6BFC31/5F6CC2BE" Ref="R?"  Part="1"
-F 0 "R?" H 3918 3896 50  0000 L CNN
+AR Path="/5F6BFC31/5F6CC2BE" Ref="R19"  Part="1"
+F 0 "R19" H 3918 3896 50  0000 L CNN
 F 1 "2.7k" H 3918 3805 50  0000 L CNN
 F 2 "" V 3890 3840 50  0001 C CNN
@@
 P 4200 3950
 AR Path="/5F6CC2C4" Ref="R?"  Part="1"
-AR Path="/5F6BFC31/5F6CC2C4" Ref="R?"  Part="1"
-F 0 "R?" H 4268 3996 50  0000 L CNN
+AR Path="/5F6BFC31/5F6CC2C4" Ref="R20"  Part="1"
+F 0 "R20" H 4268 3996 50  0000 L CNN
 F 1 "2.7k" H 4268 3905 50  0000 L CNN
 F 2 "" V 4240 3940 50  0001 C CNN
@@
 P 4100 2650
 AR Path="/5F6CC2CA" Ref="C?"  Part="1"
-AR Path="/5F6BFC31/5F6CC2CA" Ref="C?"  Part="1"
-F 0 "C?" H 4215 2696 50  0000 L CNN
+AR Path="/5F6BFC31/5F6CC2CA" Ref="C1"  Part="1"
+F 0 "C1" H 4215 2696 50  0000 L CNN
 F 1 "1uF" H 4215 2605 50  0000 L CNN
 F 2 "" H 4138 2500 50  0001 C CNN
@@
 P 3850 2350
 AR Path="/5F6CC2D0" Ref="#PWR?"  Part="1"
-AR Path="/5F6BFC31/5F6CC2D0" Ref="#PWR?"  Part="1"
-F 0 "#PWR?" H 3850 2100 50  0001 C CNN
+AR Path="/5F6BFC31/5F6CC2D0" Ref="#PWR0126"  Part="1"
+F 0 "#PWR0126" H 3850 2100 50  0001 C CNN
 F 1 "GND" H 3855 2177 50  0000 C CNN
 F 2 "" H 3850 2350 50  0001 C CNN
@@
 P 3600 3550
 AR Path="/5F6CC2D6" Ref="R?"  Part="1"
-AR Path="/5F6BFC31/5F6CC2D6" Ref="R?"  Part="1"
-F 0 "R?" V 3805 3550 50  0000 C CNN
+AR Path="/5F6BFC31/5F6CC2D6" Ref="R18"  Part="1"
+F 0 "R18" V 3805 3550 50  0000 C CNN
 F 1 "1.5k" V 3714 3550 50  0000 C CNN
 F 2 "" V 3640 3540 50  0001 C CNN
@@
 P 4300 3350
 AR Path="/5F6CC2DC" Ref="#PWR?"  Part="1"
-AR Path="/5F6BFC31/5F6CC2DC" Ref="#PWR?"  Part="1"
-F 0 "#PWR?" H 4300 3100 50  0001 C CNN
+AR Path="/5F6BFC31/5F6CC2DC" Ref="#PWR0127"  Part="1"
+F 0 "#PWR0127" H 4300 3100 50  0001 C CNN
 F 1 "GND" V 4305 3222 50  0000 R CNN
 F 2 "" H 4300 3350 50  0001 C CNN
@@
 P 3450 3550
 AR Path="/5F6CC2F0" Ref="#PWR?"  Part="1"
-AR Path="/5F6BFC31/5F6CC2F0" Ref="#PWR?"  Part="1"
-F 0 "#PWR?" H 3450 3400 50  0001 C CNN
+AR Path="/5F6BFC31/5F6CC2F0" Ref="#PWR0128"  Part="1"
+F 0 "#PWR0128" H 3450 3400 50  0001 C CNN
 F 1 "+5V" V 3465 3678 50  0000 L CNN
 F 2 "" H 3450 3550 50  0001 C CNN
@@
 P 4000 4450
 AR Path="/5F6CC2F6" Ref="#PWR?"  Part="1"
-AR Path="/5F6BFC31/5F6CC2F6" Ref="#PWR?"  Part="1"
-F 0 "#PWR?" H 4000 4300 50  0001 C CNN
+AR Path="/5F6BFC31/5F6CC2F6" Ref="#PWR0129"  Part="1"
+F 0 "#PWR0129" H 4000 4300 50  0001 C CNN
 F 1 "+5V" H 4015 4623 50  0000 C CNN
 F 2 "" H 4000 4450 50  0001 C CNN
@@
 P 4700 2650
 AR Path="/5F6CC307" Ref="C?"  Part="1"
-AR Path="/5F6BFC31/5F6CC307" Ref="C?"  Part="1"
-F 0 "C?" H 4815 2696 50  0000 L CNN
+AR Path="/5F6BFC31/5F6CC307" Ref="C2"  Part="1"
+F 0 "C2" H 4815 2696 50  0000 L CNN
 F 1 "4.7uF" H 4815 2605 50  0000 L CNN
 F 2 "" H 4738 2500 50  0001 C CNN
@@
 P 4500 2350
 AR Path="/5F6CC30D" Ref="#PWR?"  Part="1"
-AR Path="/5F6BFC31/5F6CC30D" Ref="#PWR?"  Part="1"
-F 0 "#PWR?" H 4500 2100 50  0001 C CNN
+AR Path="/5F6BFC31/5F6CC30D" Ref="#PWR0130"  Part="1"
+F 0 "#PWR0130" H 4500 2100 50  0001 C CNN
 F 1 "GND" H 4505 2177 50  0000 C CNN
 F 2 "" H 4500 2350 50  0001 C CNN
@@
 P 7400 3700
 AR Path="/5F6CC314" Ref="#PWR?"  Part="1"
-AR Path="/5F6BFC31/5F6CC314" Ref="#PWR?"  Part="1"
-F 0 "#PWR?" H 7400 3550 50  0001 C CNN
+AR Path="/5F6BFC31/5F6CC314" Ref="#PWR0131"  Part="1"
+F 0 "#PWR0131" H 7400 3550 50  0001 C CNN
 F 1 "+5V" V 7415 3828 50  0000 L CNN
 F 2 "" H 7400 3700 50  0001 C CNN
@@
 P 4500 2900
 AR Path="/5F6CC31B" Ref="#PWR?"  Part="1"
-AR Path="/5F6BFC31/5F6CC31B" Ref="#PWR?"  Part="1"
-F 0 "#PWR?" H 4500 2750 50  0001 C CNN
+AR Path="/5F6BFC31/5F6CC31B" Ref="#PWR0132"  Part="1"
+F 0 "#PWR0132" H 4500 2750 50  0001 C CNN
 F 1 "+5V" V 4515 3028 50  0000 L CNN
 F 2 "" H 4500 2900 50  0001 C CNN
@@
 P 7200 3500
 AR Path="/5F6CC32B" Ref="#PWR?"  Part="1"
-AR Path="/5F6BFC31/5F6CC32B" Ref="#PWR?"  Part="1"
-F 0 "#PWR?" H 7200 3250 50  0001 C CNN
+AR Path="/5F6BFC31/5F6CC32B" Ref="#PWR0133"  Part="1"
+F 0 "#PWR0133" H 7200 3250 50  0001 C CNN
 F 1 "GND" V 7205 3372 50  0000 R CNN
 F 2 "" H 7200 3500 50  0001 C CNN
@@
 P 3900 3550
 AR Path="/5F6CC333" Ref="D?"  Part="1"
-AR Path="/5F6BFC31/5F6CC333" Ref="D?"  Part="1"
-F 0 "D?" H 3893 3295 50  0000 C CNN
+AR Path="/5F6BFC31/5F6CC333" Ref="D17"  Part="1"
+F 0 "D17" H 3893 3295 50  0000 C CNN
 F 1 "LED" H 3893 3386 50  0000 C CNN
 F 2 "" H 3900 3550 50  0001 C CNN
@@
 P 7050 3400
 AR Path="/5F6CC33B" Ref="#PWR?"  Part="1"
-AR Path="/5F6BFC31/5F6CC33B" Ref="#PWR?"  Part="1"
-F 0 "#PWR?" H 7050 3250 50  0001 C CNN
+AR Path="/5F6BFC31/5F6CC33B" Ref="#PWR0134"  Part="1"
+F 0 "#PWR0134" H 7050 3250 50  0001 C CNN
 F 1 "+5V" V 7065 3528 50  0000 L CNN
 F 2 "" H 7050 3400 50  0001 C CNN
@@
 P 7700 2450
 AR Path="/5F6CC347" Ref="#PWR?"  Part="1"
-AR Path="/5F6BFC31/5F6CC347" Ref="#PWR?"  Part="1"
-F 0 "#PWR?" H 7700 2200 50  0001 C CNN
+AR Path="/5F6BFC31/5F6CC347" Ref="#PWR0135"  Part="1"
+F 0 "#PWR0135" H 7700 2200 50  0001 C CNN
 F 1 "GND" H 7705 2277 50  0000 C CNN
 F 2 "" H 7700 2450 50  0001 C CNN
@@
 P 7900 2600
 AR Path="/5F6CC34D" Ref="R?"  Part="1"
-AR Path="/5F6BFC31/5F6CC34D" Ref="R?"  Part="1"
-F 0 "R?" H 7832 2554 50  0000 R CNN
+AR Path="/5F6BFC31/5F6CC34D" Ref="R22"  Part="1"
+F 0 "R22" H 7832 2554 50  0000 R CNN
 F 1 "620" H 7832 2645 50  0000 R CNN
 F 2 "" V 7940 2590 50  0001 C CNN
@@
 P 8050 2900
 AR Path="/5F6CC354" Ref="R?"  Part="1"
-AR Path="/5F6BFC31/5F6CC354" Ref="R?"  Part="1"
-F 0 "R?" H 7982 2854 50  0000 R CNN
+AR Path="/5F6BFC31/5F6CC354" Ref="R24"  Part="1"
+F 0 "R24" H 7982 2854 50  0000 R CNN
 F 1 "110" H 7982 2945 50  0000 R CNN
 F 2 "" V 8090 2890 50  0001 C CNN
@@
 P 7700 3450
 AR Path="/5F6CC35B" Ref="#PWR?"  Part="1"
-AR Path="/5F6BFC31/5F6CC35B" Ref="#PWR?"  Part="1"
-F 0 "#PWR?" H 7700 3300 50  0001 C CNN
+AR Path="/5F6BFC31/5F6CC35B" Ref="#PWR0136"  Part="1"
+F 0 "#PWR0136" H 7700 3300 50  0001 C CNN
 F 1 "+5V" V 7715 3578 50  0000 L CNN
 F 2 "" H 7700 3450 50  0001 C CNN
@@
 P 7900 3200
 AR Path="/5F6CC361" Ref="R?"  Part="1"
-AR Path="/5F6BFC31/5F6CC361" Ref="R?"  Part="1"
-F 0 "R?" H 7832 3154 50  0000 R CNN
+AR Path="/5F6BFC31/5F6CC361" Ref="R23"  Part="1"
+F 0 "R23" H 7832 3154 50  0000 R CNN
 F 1 "620" H 7832 3245 50  0000 R CNN
 F 2 "" V 7940 3190 50  0001 C CNN
@@
 P 4700 3100
 AR Path="/5F6CC378" Ref="U?"  Part="1"
-AR Path="/5F6BFC31/5F6CC378" Ref="U?"  Part="1"
-F 0 "U?" H 5700 3487 60  0000 C CNN
+AR Path="/5F6BFC31/5F6CC378" Ref="U3"  Part="1"
+F 0 "U3" H 5700 3487 60  0000 C CNN
 F 1 "LTC4331IUFD-PBF" H 5700 3381 60  0000 C CNN
 F 2 "QFN_20_ADI" H 5700 3340 60  0001 C CNN
@@
 P 3850 2900
 AR Path="/5F6CC323" Ref="#PWR?"  Part="1"
-AR Path="/5F6BFC31/5F6CC323" Ref="#PWR?"  Part="1"
-F 0 "#PWR?" H 3850 2750 50  0001 C CNN
+AR Path="/5F6BFC31/5F6CC323" Ref="#PWR0137"  Part="1"
+F 0 "#PWR0137" H 3850 2750 50  0001 C CNN
 F 1 "+5V" V 3865 3028 50  0000 L CNN
 F 2 "" H 3850 2900 50  0001 C CNN
@@
 P 2350 3300
 AR Path="/5F6CC2A0" Ref="A?"  Part="1"
-AR Path="/5F6BFC31/5F6CC2A0" Ref="A?"  Part="1"
-F 0 "A?" H 2350 4481 50  0000 C CNN
+AR Path="/5F6BFC31/5F6CC2A0" Ref="A1"  Part="1"
+F 0 "A1" H 2350 4481 50  0000 C CNN
 F 1 "Arduino_UNO_R2" H 2350 4390 50  0000 C CNN
 F 2 "Module:Arduino_UNO_R2" H 2350 3300 50  0001 C CIN
@@
 P 2850 2300
 AR Path="/5F6CC2E2" Ref="#PWR?"  Part="1"
-AR Path="/5F6BFC31/5F6CC2E2" Ref="#PWR?"  Part="1"
-F 0 "#PWR?" H 2850 2150 50  0001 C CNN
+AR Path="/5F6BFC31/5F6CC2E2" Ref="#PWR0138"  Part="1"
+F 0 "#PWR0138" H 2850 2150 50  0001 C CNN
 F 1 "+5V" V 2865 2428 50  0000 L CNN
 F 2 "" H 2850 2300 50  0001 C CNN
@@
 P 6700 4100
 AR Path="/5F7519CB" Ref="#PWR?"  Part="1"
-AR Path="/5F6BFC31/5F7519CB" Ref="#PWR?"  Part="1"
-F 0 "#PWR?" H 6700 3850 50  0001 C CNN
+AR Path="/5F6BFC31/5F7519CB" Ref="#PWR0139"  Part="1"
+F 0 "#PWR0139" H 6700 3850 50  0001 C CNN
 F 1 "GND" V 6705 3972 50  0000 R CNN
 F 2 "" H 6700 4100 50  0001 C CNN
