File: ControlsPCB.sch (KiCad schematic (older format))
At the start: 7 parts, among them J1 8P8C_Shielded, J2 8P8C_Shielded, U1 LM2596S-ADJ, U3 LM2596S-ADJ

Commit message: Added 5V connection on ethernet
Connections:
- net at J1.7: now also J2.7
Changed lines of the file:
@@
+	1    0    0    -1
+$EndComp
+Wire Wire Line
+	5150 5600 7150 5600
+$Comp
+L power:+5V #PWR?
+U 1 1 5F9AF356
+P 5300 5600
+F 0 "#PWR?" H 5300 5450 50  0001 C CNN
+F 1 "+5V" H 5315 5773 50  0000 C CNN
+F 2 "" H 5300 5600 50  0001 C CNN
+F 3 "" H 5300 5600 50  0001 C CNN
+	1    5300 5600
+	1    0    0    -1
+$EndComp
+$Comp
+L power:+5V #PWR?
+U 1 1 5F9B0051
+P 6950 5600
+F 0 "#PWR?" H 6950 5450 50  0001 C CNN
+F 1 "+5V" H 6965 5773 50  0000 C CNN
+F 2 "" H 6950 5600 50  0001 C CNN
+F 3 "" H 6950 5600 50  0001 C CNN
+	1    6950 5600
 	1    0    0    -1
 $EndComp
